File: PWM.sch (KiCad schematic (older format))
At the start: 77 parts, among them J1 Conn_01x06_Male, J10 Audio-Jack-1, J11 Audio-Jack-1, J12 Audio-Jack-1, J13 Audio-Jack-1, J14 Audio-Jack-1, J15 Audio-Jack-1, J16 Audio-Jack-1, J17 Audio-Jack-1, J18 Audio-Jack-1, J19 Audio-Jack-1, J2 Jumper, J20 Audio-Jack-1, J21 Audio-Jack-1, J22 Audio-Jack-1, J23 Audio-Jack-1, J3 Jumper, J4 Jumper, J5 Jumper, J6 Jumper, J7 Jumper, J8 Audio-Jack-1, J9 Audio-Jack-1, Q1 2N3904, Q10 2N3904, Q11 2N3904, Q12 2N3904, Q13 2N3904, Q14 2N3904, Q15 2N3904, Q16 2N3904, Q2 2N3904, Q3 2N3904, Q4 2N3904, Q5 2N3904, Q6 2N3904, Q7 2N3904, Q8 2N3904, Q9 2N3904, U1 PCA9685PW, U2 uA7810

Commit message: Add files via upload
Parts:
- C2: Available (none) -> https://www.mouser.at/ProductDetail/kemet/mmk5104j50j01tr18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; MPN (none) -> MMK5104J50J01TR18L16.5TR18
- C3: Available https://www.mouser.at/ProductDetail/Murata-Electronics/RDER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 -> https://www.mouser.at/ProductDetail/kemet/mmk5104j50j01tr18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; MPN RDER71H104K0M1H03A -> MMK5104J50J01TR18L16.5TR18
- J10, J11, J12, J20, J21, J22, J23, J8, J9: Availabilty https://www.mouser.at/ProductDetail/CUI/RCJ-041?qs=%2fha2py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 -> (none); Available (none) -> https://www.mouser.at/ProductDetail/CUI/MJ1-2503A?qs=%2fha2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; MPN RCJ-041 -> MJ1-2503A
- J13, J14, J15, J16, J18, J19: Availability https://www.mouser.at/ProductDetail/CUI/RCJ-041?qs=%2fha2py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 -> (none); Available (none) -> https://www.mouser.at/ProductDetail/CUI/MJ1-2503A?qs=%2fha2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; MPN RCJ-041 -> MJ1-2503A
- J17: Available (none) -> https://www.mouser.at/ProductDetail/CUI/MJ1-2503A?qs=%2fha2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; MPN RCJ-041 -> MJ1-2503A
- J2, J3, J4, J6, J7: Available N/A -> Integrated in PCB design
- J5: Available (none) -> Integrated in PCB design
- Q1, Q10, Q11, Q12, Q13, Q14, Q15, Q16, Q2, Q3, Q4, Q5, Q6, Q7, Q8, Q9: footprint Package_TO_SOT_THT:TO-92_Inline -> TO_SOT_Packages_THT:TO-92_Inline_Narrow_Oval; Available (none) -> https://www.mouser.at/ProductDetail/Central-Semiconductor/2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; MPN (none) -> 2N3904
- R10, R11, R12, R13, R14, R15, R16, R18, R20, R22, R24, R26, R28, R30, R32, R9: Availability https://www.mouser.at/ProductDetail/Yageo/FMP200JR-52-1K?qs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 -> (none); Available (none) -> https://www.mouser.at/ProductDetail/Yageo/FMP200JR-52-1K?qs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
- RN1: Available Use standard 4K7 - 10K resistors -> Alternatively use standard 4K7 - 10K resistors
