File: PWM.kicad_pcb (KiCad board)
At the start: 2 copper layers, 85 x 56 mm, 81 parts, among them J1 Conn_01x06_Male, J10 14, J11 13, J12 1, J13 2, J14 3, J15 4, J16 5, J17 6, J18 7, J19 8, J2 Jumper, J20 12, J21 11, J22 10, J23 9, J3 Jumper, J4 Jumper, J5 Jumper, J6 Jumper, J7 Jumper, J8 16, J9 15, Q1 2N3904, Q10 2N3904, Q11 2N3904, Q12 2N3904, Q13 2N3904, Q14 2N3904, Q15 2N3904, Q16 2N3904, Q2 2N3904, Q3 2N3904, Q4 2N3904, Q5 2N3904, Q6 2N3904, Q7 2N3904, Q8 2N3904, Q9 2N3904, U1 PCA9685PW, U2 uA7810

Commit message: BOM and housing parameters updated
Parts:
- J10: value 14 -> Audio-Jack-1
- J11: value 13 -> Audio-Jack-1
- J12: value 1 -> Audio-Jack-1
- J13: value 2 -> Audio-Jack-1
- J14: value 3 -> Audio-Jack-1
- J15: value 4 -> Audio-Jack-1
- J16: value 5 -> Audio-Jack-1
- J17: value 6 -> Audio-Jack-1
- J18: value 7 -> Audio-Jack-1
- J19: value 8 -> Audio-Jack-1
- J20: value 12 -> Audio-Jack-1
- J21: value 11 -> Audio-Jack-1
- J22: value 10 -> Audio-Jack-1
- J23: value 9 -> Audio-Jack-1
- J8: value 16 -> Audio-Jack-1
- J9: value 15 -> Audio-Jack-1
- moved Q1 2.50 mm to (138.0, 108.8), turned to 90 degrees
- moved Q10 2.50 mm to (113.0, 103.5), turned to 0 degrees
- moved Q11 2.50 mm to (107.2, 103.5), turned to 0 degrees
- moved Q12 2.50 mm to (101.5, 103.5), turned to 0 degrees
- moved Q13 2.50 mm to (95.8, 103.5), turned to 0 degrees
- moved Q14 2.50 mm to (90.0, 103.5), turned to 0 degrees
- moved Q15 2.50 mm to (84.2, 103.5), turned to 0 degrees
- moved Q16 2.50 mm to (78.5, 103.5), turned to 0 degrees
- moved Q2 2.50 mm to (138.0, 103.0), turned to 90 degrees
- moved Q3 2.50 mm to (138.0, 97.2), turned to 90 degrees
- moved Q4 2.50 mm to (138.0, 91.5), turned to 90 degrees
- moved Q5 2.50 mm to (138.0, 85.8), turned to 90 degrees
- moved Q6 2.50 mm to (138.0, 80.0), turned to 90 degrees
- moved Q7 2.50 mm to (138.0, 74.2), turned to 90 degrees
- moved Q8 2.50 mm to (138.0, 68.5), turned to 90 degrees
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Connections:
- Q1 pad 1: Net-(J12-Pad2) -> GND
- Q1 pad 3: GND -> Net-(J12-Pad2)
- Q10 pad 1: Net-(J9-Pad2) -> GND
- Q10 pad 3: GND -> Net-(J9-Pad2)
- Q11 pad 1: Net-(J10-Pad2) -> GND
- Q11 pad 3: GND -> Net-(J10-Pad2)
- Q12 pad 1: Net-(J11-Pad2) -> GND
- Q12 pad 3: GND -> Net-(J11-Pad2)
- Q13 pad 1: Net-(J20-Pad2) -> GND
- Q13 pad 3: GND -> Net-(J20-Pad2)
- Q14 pad 1: Net-(J21-Pad2) -> GND
- Q14 pad 3: GND -> Net-(J21-Pad2)
- Q15 pad 1: Net-(J22-Pad2) -> GND
- Q15 pad 3: GND -> Net-(J22-Pad2)
- Q16 pad 1: Net-(J23-Pad2) -> GND
- Q16 pad 3: GND -> Net-(J23-Pad2)
- Q2 pad 1: Net-(J13-Pad2) -> GND
- Q2 pad 3: GND -> Net-(J13-Pad2)
- Q3 pad 1: Net-(J14-Pad2) -> GND
- Q3 pad 3: GND -> Net-(J14-Pad2)
- Q4 pad 1: Net-(J15-Pad2) -> GND
- Q4 pad 3: GND -> Net-(J15-Pad2)
- Q5 pad 1: Net-(J16-Pad2) -> GND
- Q5 pad 3: GND -> Net-(J16-Pad2)
- Q6 pad 1: Net-(J17-Pad2) -> GND
- Q6 pad 3: GND -> Net-(J17-Pad2)
- Q7 pad 1: Net-(J18-Pad2) -> GND
- Q7 pad 3: GND -> Net-(J18-Pad2)
- Q8 pad 1: Net-(J19-Pad2) -> GND
- Q8 pad 3: GND -> Net-(J19-Pad2)
- Q9 pad 1: Net-(J8-Pad2) -> GND
- Q9 pad 3: GND -> Net-(J8-Pad2)
